Commit message: Fix simulation

File: universal_robot/summer/summer_description/urdf/summer_hand_robot.urdf.xacro (robot description, xacro)
@@ -48,17 +48,3 @@
     <origin rpy="0 0 ${-pi/2.0}" xyz="0.051 0 0"/>
   </xacro:robotiq-3f-gripper_articulated>
-  <gazebo>
-    <!-- plugin for left RobotiQ hand -->
-    <plugin name="left_robotiq_hand_plugin" filename="libRobotiqHandPlugin.so">
-      <side>left</side>
-      <kp_position>10.0</kp_position>
-      <kd_position>0.5</kd_position>
-    </plugin>
-    <!-- plugin for right RobotiQ hand -->
-    <plugin name="right_robotiq_hand_plugin" filename="libRobotiqHandPlugin.so">
-      <side>right</side>
-      <kp_position>10.0</kp_position>
-      <kd_position>0.5</kd_position>
-    </plugin>
-  </gazebo>
 </robot>

File: universal_robot/ur_description/urdf/ur5.urdf.xacro (robot description, xacro)
@@ -19,4 +19,6 @@
      wrist_2_lower_limit:=${-pi}    wrist_2_upper_limit:=${pi}
      wrist_3_lower_limit:=${-pi}    wrist_3_upper_limit:=${pi}">
+    <!-- friction-->
+    <xacro:property name="arm_friction" value="1" />
     <!-- Inertia parameters -->
     <xacro:property name="base_mass" value="4.0" />  <!-- This mass might be incorrect -->
@@ -103,5 +105,5 @@
         <limit lower="${shoulder_pan_lower_limit}" upper="${shoulder_pan_upper_limit}" effort="150.0" velocity="3.15"/>
       </xacro:if>
-      <dynamics damping="0.0" friction="0.0"/>
+      <dynamics damping="0.0" friction="${arm_friction}"/>
     </joint>
     <link name="${prefix}shoulder_link">
@@ -134,5 +136,5 @@
         <limit lower="${shoulder_lift_lower_limit}" upper="${shoulder_lift_upper_limit}" effort="150.0" velocity="3.15"/>
       </xacro:if>
-      <dynamics damping="0.0" friction="0.0"/>
+      <dynamics damping="0.0" friction="${arm_friction}"/>
     </joint>
     <link name="${prefix}upper_arm_link">
@@ -165,5 +167,5 @@
         <limit lower="${elbow_joint_lower_limit}" upper="${elbow_joint_upper_limit}" effort="150.0" velocity="3.15"/>
       </xacro:if>
-      <dynamics damping="0.0" friction="0.0"/>
+      <dynamics damping="0.0" friction="${arm_friction}"/>
     </joint>
     <link name="${prefix}forearm_link">
@@ -196,5 +198,5 @@
         <limit lower="${wrist_1_lower_limit}" upper="${wrist_1_upper_limit}" effort="28.0" velocity="3.2"/>
       </xacro:if>
-      <dynamics damping="0.0" friction="0.0"/>
+      <dynamics damping="0.0" friction="${arm_friction}"/>
     </joint>
     <link name="${prefix}wrist_1_link">
@@ -227,5 +229,5 @@
         <limit lower="${wrist_2_lower_limit}" upper="${wrist_2_upper_limit}" effort="28.0" velocity="3.2"/>
       </xacro:if>
-      <dynamics damping="0.0" friction="0.0"/>
+      <dynamics damping="0.0" friction="${arm_friction}"/>
     </joint>
     <link name="${prefix}wrist_2_link">
@@ -258,5 +260,5 @@
         <limit lower="${wrist_3_lower_limit}" upper="${wrist_3_upper_limit}" effort="28.0" velocity="3.2"/>
       </xacro:if>
-      <dynamics damping="0.0" friction="0.0"/>
+      <dynamics damping="0.0" friction="${arm_friction}"/>
     </joint>
     <link name="${prefix}wrist_3_link">
